File: KiCad Projects/ADC_and_amplifier_pico_breakout_board/_restore_backup_2026-08-18T02-27-18-975/ADC_and_amplifier_pico_breakout_board.kicad_sch (KiCad schematic)
At the start: 66 parts, among them J1 SMA_KWE_THT, J2 Pimoroni_Pico_LiPo_2_XL_W, U1 MAX5394LATA+T, U2 SN74AHCT125DRG4, U3 OPA365xxDBV, U4 OPA365xxDBV, U5 AD9226ARSRL, U6 AD8138AR-REEL

Commit message: Finished the PCB for the ADC and AMP board
Parts:
- removed TP1: SPI_CS, TestPoint:TestPoint_Loop_D2.50mm_Drill1.0mm, symbol Connector:TestPoint
- removed TP10: ADC OTR, TestPoint:TestPoint_Loop_D2.50mm_Drill1.0mm, symbol Connector:TestPoint
- removed TP11: ADC 2.5V, TestPoint:TestPoint_Loop_D2.50mm_Drill1.0mm, symbol Connector:TestPoint
- removed TP12: ADC VREF, TestPoint:TestPoint_Loop_D2.50mm_Drill1.0mm, symbol Connector:TestPoint
- removed TP13: ADC_CLK, TestPoint:TestPoint_Loop_D2.50mm_Drill1.0mm, symbol Connector:TestPoint
- removed TP14: SIG_FILTERED, TestPoint:TestPoint_Loop_D2.50mm_Drill1.0mm, symbol Connector:TestPoint
- removed TP2: AMP1_OUT, TestPoint:TestPoint_Loop_D2.50mm_Drill1.0mm, symbol Connector:TestPoint
- removed TP3: AMP2_IN, TestPoint:TestPoint_Loop_D2.50mm_Drill1.0mm, symbol Connector:TestPoint
- removed TP4: AMP2_OUT, TestPoint:TestPoint_Loop_D2.50mm_Drill1.0mm, symbol Connector:TestPoint
- removed TP5: TP_GND1, TestPoint:TestPoint_Loop_D2.50mm_Drill1.0mm, symbol Connector:TestPoint
- removed TP6: TP_GND2, TestPoint:TestPoint_Loop_D2.50mm_Drill1.0mm, symbol Connector:TestPoint
- removed TP7: 5VA, TestPoint:TestPoint_Loop_D2.50mm_Drill1.0mm, symbol Connector:TestPoint
- removed TP8: DIGIPOT_2.5V, TestPoint:TestPoint_Loop_D2.50mm_Drill1.0mm, symbol Connector:TestPoint
- removed TP9: SIG_2.5V, TestPoint:TestPoint_Loop_D2.50mm_Drill1.0mm, symbol Connector:TestPoint
- removed U2: SN74AHCT125DRG4, ul_SN74AHCT125DRG4:D14_TEX, symbol ul_SN74AHCT125DRG4:SN74AHCT125DRG4
- added C21: 100nF, Capacitor_SMD:C_1206_3216Metric, symbol Device:C
- added U2: 74AHCT125D_118, SO14_SOT108-1_NEX, symbol ul_74AHCT125D-118:74AHCT125D_118
Connections:
- net +3.3V: now also C21.1
- net +5V: now also U2.14 (VCC)
- net GND: now also C21.2, U2.1 (1OE), U2.10 (3OE), U2.12 (4A), U2.13 (4OE), U2.4 (2OE), U2.7 (GND); no longer J2.03 (GND), J2.08 (GND), J2.13 (GND), J2.18 (GND), J2.23 (GND), J2.28 (GND), J2.33 (GND), J2.38 (GND), J2.43 (GND), J2.48 (GND), J2.53 (GND), J2.58 (GND)
- net at J2.19 (GP14_SCK): now also U2.2 (1A)
- net at U1.5 (SCLK): now also U2.3 (1Y)
- net at J2.20 (GP15_TX): now also U2.5 (2A)
- net at U1.4 (DIN): now also U2.6 (2Y)
- net at U1.3 (*CS): now also U2.8 (3Y)
- net at J2.17 (GP13_CSn): now also U2.9 (3A)
Other:
- moved on the sheet: C20, D3, FB1, R4
