File: KiCad Projects/ADC_AMP_with_MCP4161/ADC_AMP_with_MCP4161.kicad_pcb (KiCad board)
At the start: 4 copper layers, 55 x 80.5 mm, 70 parts, among them J1 SMA_KWE_THT, J2 Pimoroni_Pico_LiPo_2_XL_W, U1 MAX5394LATA+T, U2 SN74AHCT125DRG4, U3 OPA365xxDBV, U4 OPA365xxDBV, U5 AD9226ARSRL, U6 AD8138AR-REEL

Commit message: Finished the PCB for the ADC and AMP board
Parts:
- removed U1: MAX5394LATA+T, MAX5394:21-0168_T822-2_MXM
- added U7: MCP4161T-502E/SN, MCP4161T-502ESN:SOIC8-N_MC_MCH, F.Cu at (164.8, 88.5)
- moved C9 11.2 mm to (168.0, 93.5), turned to 0 degrees
- moved R6 7.91 mm to (164.3, 98.8), turned to 0 degrees
- moved C10 6.59 mm to (163.8, 93.2), turned to 0 degrees
- moved C3 5.55 mm to (161.4, 99.5)
- moved C12 5.50 mm to (158.2, 99.8)
- moved C16 5.50 mm to (162.1, 106.7)
- moved D1 5.50 mm to (163.0, 104.8)
- moved D2 5.50 mm to (163.0, 102.2)
- moved R1 5.50 mm to (161.4, 109.2)
- moved R12 5.50 mm to (156.2, 100.3)
- moved R13 5.50 mm to (156.2, 97.2)
- moved R2 5.50 mm to (159.2, 97.2)
- moved U3 5.50 mm to (163.2, 96.2)
- moved R8 5.34 mm to (168.7, 101.5), turned to 180 degrees
- moved C5 4.86 mm to (167.8, 96.0), turned to 180 degrees
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Connections:
- C9 pad 1: GND -> +5V
- C9 pad 2: +5V -> GND
Routing:
- net Net-(U7-P0A): track 43.3 -> 25.4 mm
- net +5V: track 151.9 -> 166.3 mm, vias 8 -> 7
- net Net-(C12-Pad2): track 19.0 -> 11.5 mm
- net Net-(J1-SIGNAL): track 17.4 -> 11.9 mm
- net Net-(U2-1Y): track 10.5 -> 14.7 mm
- net Net-(U2-3Y): track 39.9 -> 35.8 mm
- net Net-(U3-+): track 24.5 -> 20.5 mm
- net Net-(U3--): track 7.64 -> 3.84 mm
- net GND: track 73.1 -> 75.7 mm
- net Net-(U7-P0B): track 49.0 -> 47.1 mm
- net Net-(U4-+): track 17.7 -> 19.5 mm
- net Net-(J2-GP15_TX): track 35.2 -> 33.8 mm
- net Net-(U2-2Y): track 7.94 -> 6.84 mm
Other:
- board text added: "*"
- board text added: "OPA365 (U3, U4) MCP4161-503 (U7) AD8138 (U6) ADC9226 (U5)"

Commit message: a couple more small changes
Parts:
- added C21: 100nF, Capacitor_SMD:C_1206_3216Metric, F.Cu at (160.4, 52.1)
- added D4: LED, LED_SMD:LED_0603_1608Metric, F.Cu at (172.5, 103.2)
- added R15: 470, Resistor_SMD:R_0603_1608Metric, F.Cu at (169.2, 103.2)
- moved R4 12.7 mm to (168.8, 49.4), turned to -90 degrees
- moved D3 8.85 mm to (168.8, 52.6), turned to -90 degrees
Connections:
- J2 pad 22: unconnected-(J2-GP31_TX-Pad22) -> Net-(D4-A)
Routing:
- net GND: track 75.7 -> 79.9 mm, vias 28 -> 29
- net +5V: track 166.3 -> 163.4 mm, vias 7 -> 8
- net Net-(D3-A): track 22.8 -> 25.8 mm
- net Net-(D4-A): track 0.00 -> 2.94 mm
- net Net-(U4-+): track 19.5 -> 21.4 mm
- net Net-(D4-K): track 0.00 -> 1.64 mm
Other:
- board text added: "+5V OK"
- board text added: "2.5V FLOAT"
- board text added: "Heartbeat LED"
- board text added: "v1.0 2026-08-19 Designed by Will Martin"
- board text removed: "SIG ON 2.5V"
- board text removed: "v1.0 Signed On 2026-08-19"
