File: KiCad Projects/ADC_AMP_with_MCP4161/ADC_AMP_with_MCP4161.kicad_sch (KiCad schematic)
At the start: 66 parts, among them J1 SMA_KWE_THT, J2 Pimoroni_Pico_LiPo_2_XL_W, U1 MAX5394LATA+T, U2 SN74AHCT125DRG4, U3 OPA365xxDBV, U4 OPA365xxDBV, U5 AD9226ARSRL, U6 AD8138AR-REEL

Commit message: Finished the PCB for the ADC and AMP board
Parts:
- removed U1: MAX5394LATA+T, 21-0168_T822-2_MXM, symbol MAX5394LATA:MAX5394LATA+T
- added U7: MCP4161T-502E/SN, MCP4161T-502ESN:SOIC8-N_MC_MCH, symbol MCP4161T-502ESN:MCP4161T-502E_SN
Connections:
- net +5V: now also C9.1, U7.8 (VDD); no longer C9.2
- net GND: now also C9.2, U7.4 (VSS); no longer C9.1
- net at C10.2, R10.1, R11.2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: now also U7.7 (P0B)
- net at U2.3 (1Y): now also U7.2 (SCK)
- net at U2.6 (2Y): now also U7.3 (SDI/SDO)
- net at TP1.1, U2.8 (3Y): now also U7.1 (*CS)
- net at R6.1, TP2.1, U3.1: now also U7.5 (P0A)
- net at TP3.1, U4.3 (+): now also U7.6 (P0W)
Other:
- moved on the sheet: C10, C9, R10, R11, TP1, TP8

Commit message: a couple more small changes
Parts:
- added C21: 100nF, Capacitor_SMD:C_1206_3216Metric, symbol Device:C
- added D4: LED, LED_SMD:LED_0603_1608Metric, symbol Device:LED
- added R15: 470, Resistor_SMD:R_0603_1608Metric, symbol Device:R
Connections:
- net +5V: now also C21.1
- net GND: now also C21.2, R15.1
- net at J2.22 (GP31_TX): now also D4.2 (A)
- new net: D4.1 (K), R15.2
